File: WeMos-RN2483.brd (EAGLE design)
At the start: 36.3 x 25.7 mm, 25 parts, among them P2 PADNORMAL, P3 PADNORMAL, SW1 DHT-4235A, U1 RN2483

Commit message: Version V1.1 update
Parts:
- removed R5: 10K, _c2h:0805-RES
- U$2: value LED -> GRN
- U$3: value LED -> RED
- moved U$1 3.18 mm to (24.6, 16.8)
Connections:
- net 3V3: no longer R5.2
- net GPIO12: now also U1.RESET°; no longer JTX.1
- net GPIO13: now also JTX.1; no longer JRX.3
- net GPIO14: no longer R5.1, SW1.1, SW1.2
- net GPIO15: now also JRX.3; no longer U1.RESET°
- net GPIO2: now also SW1.2
- net N$1: now also U1.GPIO1; no longer U1.GPIO0
Routing:
- net GPIO14: track 31.7 -> 0.00 mm
- net GPIO12: track 9.58 -> 26.9 mm, vias 0 -> 2
- net GPIO2: track 0.00 -> 15.6 mm
- net 3V3: track 84.5 -> 72.1 mm, vias 4 -> 3
- net GPIO15: track 21.6 -> 10.1 mm, vias 1 -> 0
- net GPIO0: track 17.9 -> 24.8 mm
- net N$2: track 2.86 -> 5.46 mm
- net GPIO13: track 9.05 -> 10.6 mm
- net UART_TX: track 9.57 -> 11.0 mm
- net N$1: track 4.60 -> 5.22 mm
Other:
- outline, holes or cut-outs redrawn
- board text added: "IO15"
- board text added: "V1.1"
- board text removed: "IO12"
- board text removed: "V1.0"
