File: WeMos-RN2483.brd (EAGLE design)
At the start: 36.3 x 25.7 mm, 24 parts, among them P2 PADNORMAL, P3 PADNORMAL, SW1 DHT-4235A, U1 RN2483

Commit message: Updated to V1.2
Routing:
- net GND: track 0.00 -> 9.19 mm, vias 61 -> 62
- net SDA: track 30.4 -> 29.2 mm
- net SCL: track 33.5 -> 33.0 mm
Other:
- board text added: "V1.2"
- board text removed: "V1.1"
Changed lines of the file:
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@@
 <text x="22.09975" y="1.91025" size="1.27" layer="26" font="vector" ratio="15" rot="MR0">-</text>
 <text x="21.02025" y="1.78325" size="1.143" layer="26" font="vector" ratio="15" rot="MR0">+</text>
-<text x="5.23875" y="23.8125" size="1.4224" layer="26" font="vector" ratio="15" rot="MR0" align="center">V1.1</text>
-<text x="8.89" y="13.23975" size="1.4224" layer="25" font="vector" ratio="15" rot="R90" align="center">V1.1</text>
+<text x="5.23875" y="23.8125" size="1.4224" layer="26" font="vector" ratio="15" rot="MR0" align="center">V1.2</text>
+<text x="8.89" y="13.23975" size="1.4224" layer="25" font="vector" ratio="15" rot="R90" align="center">V1.2</text>
 <text x="6.2865" y="18.76425" size="0.889" layer="25" font="vector" ratio="15" rot="R270" align="center">433</text>
 <text x="1.016" y="21.24075" size="0.8128" layer="26" font="vector" ratio="15" rot="MR90" align="center">433 MHz</text>
@@
 </signal>
 <signal name="GND">
-<polygon width="0.254" layer="16">
+<polygon width="0.254" layer="16" isolate="0.254">
 <vertex x="37.465" y="26.67"/>
 <vertex x="37.465" y="-1.27"/>
@@
 <vertex x="-1.27" y="26.67"/>
 </polygon>
-<polygon width="0.254" layer="1">
+<polygon width="0.254" layer="1" isolate="0.254">
 <vertex x="-0.635" y="26.035"/>
 <vertex x="36.83" y="26.035"/>
@@
 <via x="6.985" y="10.16" extent="1-16" drill="0.3556" diameter="0.7112"/>
 <via x="32.385" y="21.844" extent="1-16" drill="0.3556" diameter="0.7112"/>
-<via x="19.939" y="19.1135" extent="1-16" drill="0.3556" diameter="0.7112"/>
 <via x="33.655" y="15.875" extent="1-16" drill="0.3556" diameter="0.7112"/>
 <contactref element="WS2812" pad="3"/>
@@
 <via x="10.16" y="5.715" extent="1-16" drill="0.3556" diameter="0.7112"/>
 <via x="11.43" y="5.715" extent="1-16" drill="0.3556" diameter="0.7112"/>
-<via x="11.43" y="6.985" extent="1-16" drill="0.3556" diameter="0.7112"/>
 <via x="11.43" y="8.255" extent="1-16" drill="0.3556" diameter="0.7112"/>
 <via x="11.43" y="9.525" extent="1-16" drill="0.3556" diameter="0.7112"/>
@@
 <via x="25.4" y="7.8105" extent="1-16" drill="0.3556" diameter="0.7112"/>
 <via x="23.71725" y="4.445" extent="1-16" drill="0.3556" diameter="0.7112"/>
-<via x="15.875" y="2.7305" extent="1-16" drill="0.3556" diameter="0.7112"/>
+<wire x1="14.605" y1="24.13" x2="14.986" y2="24.13" width="0.4064" layer="16"/>
+<wire x1="14.986" y1="24.13" x2="16.383" y2="22.733" width="0.4064" layer="16"/>
+<wire x1="16.383" y1="22.733" x2="16.383" y2="21.844" width="0.4064" layer="16"/>
+<wire x1="16.383" y1="21.844" x2="16.51" y2="21.717" width="0.4064" layer="16"/>
+<via x="26.797" y="19.939" extent="1-16" drill="0.3556" diameter="0.7112"/>
+<wire x1="14.605" y1="24.13" x2="14.605" y2="23.495" width="0.4064" layer="16"/>
+<wire x1="14.605" y1="23.495" x2="11.43" y2="20.32" width="0.4064" layer="16"/>
+<wire x1="11.43" y1="20.32" x2="11.43" y2="19.685" width="0.4064" layer="16"/>
+<via x="14.224" y="14.351" extent="1-16" drill="0.3556" diameter="0.7112"/>
+<via x="17.272" y="14.351" extent="1-16" drill="0.3556" diameter="0.7112"/>
+<via x="19.812" y="19.177" extent="1-16" drill="0.3556" diameter="0.7112"/>
 </signal>
 <signal name="SCL">
@@
 <wire x1="18.669" y1="13.97" x2="18.7325" y2="13.97" width="0.3048" layer="1"/>
 <wire x1="18.7325" y1="13.97" x2="23.495" y2="13.97" width="0.3048" layer="16"/>
-<wire x1="23.495" y1="13.97" x2="25.4" y2="15.875" width="0.3048" layer="16"/>
-<wire x1="25.4" y1="15.875" x2="25.4" y2="23.495" width="0.3048" layer="16"/>
-<wire x1="25.4" y1="23.495" x2="24.765" y2="24.13" width="0.3048" layer="16"/>
+<wire x1="24.765" y1="15.24" x2="23.495" y2="13.97" width="0.3048" layer="16"/>
+<wire x1="24.765" y1="24.13" x2="24.765" y2="15.24" width="0.3048" layer="16"/>
 </signal>
 <signal name="SDA">
@@
 <contactref element="I2C_OLED" pad="4"/>
 <contactref element="JP1" pad="4"/>
-<via x="20.32" y="16.51" extent="1-16" drill="0.3556" diameter="0.7112"/>
-<wire x1="20.32" y1="16.51" x2="23.495" y2="19.685" width="0.3048" layer="16"/>
+<via x="19.685" y="16.51" extent="1-16" drill="0.3556" diameter="0.7112"/>
 <wire x1="3.302" y1="16.51" x2="3.937" y2="15.875" width="0.254" layer="1"/>
 <wire x1="3.937" y1="15.875" x2="7.62" y2="15.875" width="0.254" layer="1"/>
-<wire x1="13.97" y1="13.97" x2="9.525" y2="13.97" width="0.254" layer="1"/>
-<wire x1="9.525" y1="13.97" x2="7.62" y2="15.875" width="0.254" layer="1"/>
-<wire x1="13.335" y1="12.43" x2="13.335" y2="13.335" width="0.3048" layer="1"/>
-<wire x1="13.335" y1="13.335" x2="13.97" y2="13.97" width="0.3048" layer="1"/>
-<wire x1="23.495" y1="19.685" x2="23.495" y2="22.225" width="0.3048" layer="16"/>
-<wire x1="23.495" y1="22.225" x2="22.225" y2="23.495" width="0.3048" layer="16"/>
-<wire x1="22.225" y1="23.495" x2="22.225" y2="24.13" width="0.3048" layer="16"/>
-<wire x1="13.97" y1="13.97" x2="17.145" y2="13.97" width="0.3048" layer="1"/>
-<wire x1="17.145" y1="13.97" x2="19.685" y2="16.51" width="0.3048" layer="1"/>
-<wire x1="19.685" y1="16.51" x2="20.32" y2="16.51" width="0.3048" layer="1"/>
+<wire x1="12.7" y1="15.24" x2="8.255" y2="15.24" width="0.254" layer="1"/>
+<wire x1="8.255" y1="15.24" x2="7.62" y2="15.875" width="0.254" layer="1"/>
+<wire x1="13.335" y1="12.43" x2="13.335" y2="14.605" width="0.3048" layer="1"/>
+<wire x1="13.335" y1="14.605" x2="12.7" y2="15.24" width="0.3048" layer="1"/>
+<wire x1="12.7" y1="15.24" x2="18.415" y2="15.24" width="0.3048" layer="1"/>
+<wire x1="18.415" y1="15.24" x2="19.685" y2="16.51" width="0.3048" layer="1"/>
+<wire x1="22.225" y1="24.13" x2="22.225" y2="19.05" width="0.3048" layer="16"/>
+<wire x1="22.225" y1="19.05" x2="19.685" y2="16.51" width="0.3048" layer="16"/>
 </signal>
 <signal name="GPIO14">
@@
 <wire x1="15.24" y1="21.717" x2="15.24" y2="18.669" width="0.3048" layer="16"/>
 <wire x1="15.24" y1="18.669" x2="15.8115" y2="18.0975" width="0.3048" layer="16"/>
-<via x="15.8115" y="18.0975" extent="1-16" drill="0.6"/>
+<via x="15.8115" y="18.0975" extent="1-16" drill="0.3556" diameter="0.7112"/>
 <wire x1="15.8115" y1="18.0975" x2="20.32" y2="18.0975" width="0.3048" layer="1"/>
 <wire x1="20.32" y1="18.0975" x2="21.59" y2="16.8275" width="0.3048" layer="1"/>
@@
 <via x="24.765" y="13.335" extent="1-16" drill="0.3556" diameter="0.7112"/>
 <wire x1="27.94" y1="16.51" x2="27.94" y2="23.495" width="0.3048" layer="16"/>
-<wire x1="27.94" y1="23.495" x2="27.305" y2="24.13" width="0.3048" layer="16"/>
 <wire x1="27.94" y1="16.51" x2="24.765" y2="13.335" width="0.3048" layer="16"/>
 <wire x1="23.495" y1="12.319" x2="23.495" y2="12.065" width="0.3048" layer="1"/>
 <wire x1="23.495" y1="12.065" x2="24.765" y2="13.335" width="0.3048" layer="1"/>
+<wire x1="27.94" y1="23.495" x2="27.305" y2="24.13" width="0.3048" layer="16"/>
 </signal>
 <signal name="RST">
@@
 <wire x1="19.685" y1="21.59" x2="13.335" y2="21.59" width="0.6096" layer="1"/>
 <wire x1="13.335" y1="21.59" x2="12.065" y2="22.86" width="0.6096" layer="1"/>
-<wire x1="26.67" y1="10.16" x2="26.67" y2="13.335" width="0.6096" layer="1"/>
-<wire x1="26.67" y1="13.335" x2="22.225" y2="17.78" width="0.6096" layer="1"/>
-<wire x1="22.225" y1="17.78" x2="22.225" y2="19.05" width="0.6096" layer="1"/>
-<wire x1="22.225" y1="19.05" x2="19.685" y2="21.59" width="0.6096" layer="1"/>
+<wire x1="26.67" y1="10.16" x2="26.67" y2="14.605" width="0.6096" layer="1"/>
+<wire x1="26.67" y1="14.605" x2="19.685" y2="21.59" width="0.6096" layer="1"/>
 </signal>
 <signal name="DO">
