File: WeMos-RN2483.sch (EAGLE design)
At the start: 23 parts, among them P2 PADNORMAL, P3 PADNORMAL, SW1 DHT-4235A, U1 RN2483

Commit message: Version V1.1 update
Parts:
- removed R5: 10K, _c2h:RESISTOR0805-RES
- U$2: value LED -> GRN
- U$3: value LED -> RED
Connections:
- net 3V3: no longer R5.2
- net GPIO12: now also U1.RESET°; no longer JTX.1
- net GPIO13: now also JTX.1; no longer JRX.3
- net GPIO14: no longer R5.1, SW1.A0, SW1.A1
- net GPIO15: now also JRX.3; no longer U1.RESET°
- net GPIO2: now also SW1.A1
- net N$1: now also U1.GPIO1; no longer U1.GPIO0
Other:
- note added: "WeMos already have a pullup on GPIO2"
Changed lines of the file:
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@@
 <layer number="56" name="wert" color="7" fill="1" visible="no" active="no"/>
 <layer number="57" name="tCAD" color="7" fill="1" visible="no" active="no"/>
+<layer number="58" name="b3D" color="7" fill="1" visible="no" active="no"/>
 <layer number="59" name="tCarbon" color="7" fill="1" visible="no" active="no"/>
 <layer number="60" name="bCarbon" color="7" fill="1" visible="no" active="no"/>
@@
 <part name="NAME" library="SparkFun-Aesthetics" deviceset="FRAME-A4L" device="" value="Value">
 <attribute name="CNAME" value="ESP8266 WeMos Lora RN2483 Shield"/>
-<attribute name="CREVISION" value="1.0"/>
+<attribute name="CREVISION" value="1.1"/>
 <attribute name="DESIGNER" value="Charles-Henri Hallard"/>
 </part>
@@
 <part name="R3" library="_c2h" deviceset="RESISTOR" device="0805-RES" value="390"/>
 <part name="R4" library="_c2h" deviceset="RESISTOR" device="0805-RES" value="390"/>
-<part name="U$2" library="_c2h" deviceset="LED" device="0805" value="LED"/>
-<part name="U$3" library="_c2h" deviceset="LED" device="0805" value="LED"/>
+<part name="U$2" library="_c2h" deviceset="LED" device="0805" value="GRN"/>
+<part name="U$3" library="_c2h" deviceset="LED" device="0805" value="RED"/>
 <part name="GND6" library="supply1" deviceset="GND" device=""/>
 <part name="GND7" library="supply1" deviceset="GND" device=""/>
-<part name="R5" library="_c2h" deviceset="RESISTOR" device="0805-RES" value="10K"/>
 <part name="GND10" library="supply1" deviceset="GND" device=""/>
-<part name="+3V2" library="supply1" deviceset="+3V3" device=""/>
 <part name="SW1" library="Switch-2016" deviceset="SMD-BUTTON-TOP-DHT-4235A(4P-4.2X3.2MM)" device="" value="DHT-4235A"/>
 </parts>
@@
 <text x="105.41" y="120.65" size="1.778" layer="94">433MHz</text>
 <text x="105.41" y="135.89" size="1.778" layer="94">868MHz</text>
+<text x="86.36" y="41.91" size="1.778" layer="94">WeMos already have
+a pullup on GPIO2</text>
 </plain>
 <instances>
@@
 <attribute name="VALUE" x="243.84" y="137.16" size="1.778" layer="96" rot="R180"/>
 </instance>
-<instance part="GND9" gate="1" x="114.3" y="111.76"/>
+<instance part="GND9" gate="1" x="114.3" y="99.06"/>
 <instance part="WS2812" gate="G$1" x="134.62" y="30.48" smashed="yes">
 <attribute name="NAME" x="121.92" y="36.068" size="1.6764" layer="95"/>
@@
 <instance part="GND6" gate="1" x="30.48" y="91.44"/>
 <instance part="GND7" gate="1" x="22.86" y="91.44"/>
-<instance part="R5" gate="G$1" x="85.09" y="49.53" smashed="yes" rot="R90">
-<attribute name="NAME" x="88.9254" y="48.641" size="1.778" layer="95" rot="R90"/>
-<attribute name="VALUE" x="83.82" y="48.006" size="1.778" layer="96" rot="R90"/>
-</instance>
 <instance part="GND10" gate="1" x="85.09" y="15.875"/>
-<instance part="+3V2" gate="G$1" x="85.09" y="58.42" smashed="yes">
-<attribute name="VALUE" x="87.63" y="60.96" size="1.778" layer="96" rot="R180"/>
-</instance>
 <instance part="SW1" gate="G$1" x="85.09" y="33.02"/>
 </instances>
@@
 <junction x="111.76" y="116.84"/>
 <pinref part="J$1" gate="1" pin="GND@3"/>
-<wire x1="114.3" y1="116.84" x2="114.3" y2="114.3" width="0.1524" layer="91"/>
+<wire x1="114.3" y1="116.84" x2="114.3" y2="101.6" width="0.1524" layer="91"/>
 <junction x="114.3" y="116.84"/>
 </segment>
@@
 <label x="140.97" y="133.35" size="1.778" layer="95"/>
 </segment>
-<segment>
-<pinref part="R5" gate="G$1" pin="1"/>
-<wire x1="85.09" y1="44.45" x2="85.09" y2="43.18" width="0.1524" layer="91"/>
-<wire x1="85.09" y1="43.18" x2="85.09" y2="40.64" width="0.1524" layer="91"/>
-<wire x1="85.09" y1="43.18" x2="96.52" y2="43.18" width="0.1524" layer="91"/>
-<junction x="85.09" y="43.18"/>
-<label x="87.63" y="43.18" size="1.778" layer="95"/>
-<pinref part="SW1" gate="G$1" pin="A0"/>
-<wire x1="85.09" y1="40.64" x2="76.2" y2="40.64" width="0.1524" layer="91"/>
-<wire x1="76.2" y1="40.64" x2="76.2" y2="35.56" width="0.1524" layer="91"/>
-<pinref part="SW1" gate="G$1" pin="A1"/>
-<wire x1="93.98" y1="35.56" x2="93.98" y2="40.64" width="0.1524" layer="91"/>
-<wire x1="93.98" y1="40.64" x2="85.09" y2="40.64" width="0.1524" layer="91"/>
-<junction x="85.09" y="40.64"/>
-</segment>
 </net>
 <net name="GPIO12" class="0">
@@
 <label x="140.97" y="130.81" size="1.778" layer="95"/>
 <pinref part="JP2" gate="G$1" pin="5"/>
-</segment>
-<segment>
-<pinref part="JTX" gate="G$1" pin="1"/>
-<wire x1="40.64" y1="116.84" x2="48.26" y2="116.84" width="0.1524" layer="91"/>
-<label x="40.64" y="116.84" size="1.778" layer="95"/>
-</segment>
-</net>
-<net name="GPIO13" class="0">
-<segment>
-<pinref part="JP2" gate="G$1" pin="6"/>
-<wire x1="148.59" y1="128.27" x2="140.97" y2="128.27" width="0.1524" layer="91"/>
-<label x="140.97" y="128.27" size="1.778" layer="95"/>
-</segment>
-<segment>
-<pinref part="JRX" gate="G$1" pin="3"/>
-<wire x1="40.64" y1="129.54" x2="48.26" y2="129.54" width="0.1524" layer="91"/>
-<label x="40.64" y="129.54" size="1.778" layer="95"/>
-</segment>
-</net>
-<net name="GPIO15" class="0">
-<segment>
-<pinref part="JP2" gate="G$1" pin="7"/>
-<wire x1="148.59" y1="125.73" x2="140.97" y2="125.73" width="0.1524" layer="91"/>
-<label x="140.97" y="125.73" size="1.778" layer="95"/>
 </segment>
 <segment>
@@
 <pinref part="U1" gate="G$1" pin="RESET°"/>
 <junction x="60.96" y="129.54"/>
+</segment>
+</net>
+<net name="GPIO13" class="0">
+<segment>
+<pinref part="JP2" gate="G$1" pin="6"/>
+<wire x1="148.59" y1="128.27" x2="140.97" y2="128.27" width="0.1524" layer="91"/>
+<label x="140.97" y="128.27" size="1.778" layer="95"/>
+</segment>
+<segment>
+<pinref part="JTX" gate="G$1" pin="1"/>
+<wire x1="40.64" y1="116.84" x2="48.26" y2="116.84" width="0.1524" layer="91"/>
+<label x="40.64" y="116.84" size="1.778" layer="95"/>
+</segment>
+</net>
+<net name="GPIO15" class="0">
+<segment>
+<pinref part="JP2" gate="G$1" pin="7"/>
+<wire x1="148.59" y1="125.73" x2="140.97" y2="125.73" width="0.1524" layer="91"/>
+<label x="140.97" y="125.73" size="1.778" layer="95"/>
+</segment>
+<segment>
+<pinref part="JRX" gate="G$1" pin="3"/>
+<wire x1="40.64" y1="129.54" x2="48.26" y2="129.54" width="0.1524" layer="91"/>
+<label x="40.64" y="129.54" size="1.778" layer="95"/>
 </segment>
 </net>
@@
 <wire x1="248.92" y1="49.53" x2="231.14" y2="49.53" width="0.1524" layer="91"/>
 </segment>
-<segment>
-<pinref part="+3V2" gate="G$1" pin="+3V3"/>
-<pinref part="R5" gate="G$1" pin="2"/>
-<wire x1="85.09" y1="55.88" x2="85.09" y2="54.61" width="0.1524" layer="91"/>
-</segment>
 </net>
 <net name="A0" class="0">
@@
 <wire x1="184.15" y1="128.27" x2="189.23" y2="128.27" width="0.1524" layer="91"/>
 <label x="184.15" y="128.27" size="1.778" layer="95"/>
+</segment>
+<segment>
+<wire x1="93.98" y1="35.56" x2="104.14" y2="35.56" width="0.1524" layer="91"/>
+<label x="94.996" y="36.068" size="1.778" layer="95"/>
+<pinref part="SW1" gate="G$1" pin="A1"/>
 </segment>
 </net>
@@
 <net name="N$1" class="0">
 <segment>
-<pinref part="U1" gate="G$1" pin="GPIO0"/>
+<pinref part="U1" gate="G$1" pin="GPIO1"/>
 <pinref part="R4" gate="G$1" pin="2"/>
 <wire x1="60.96" y1="109.22" x2="49.53" y2="109.22" width="0.1524" layer="91"/>
